Commit message: test pushing box, not solvable yet

File: model/urdf/ur5_robot.urdf (robot description, URDF)
Before this commit: robot ur5, 11 links, 10 joints
Links:
- link base_link: geometry collision mesh filename=/home/mzwang/catkin_ws/src/trajectory_my/model/meshes/ur5/c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; visual mesh filename=/home/mzwang/catkin_ws/src/trajectory_my/model/meshes/ur5/v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
- link forearm_link: geometry collision mesh filename=/home/mzwang/catkin_ws/src/trajectory_my/model/meshes/ur5/c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; visual mesh filename=/home/mzwang/catkin_ws/src/trajectory_my/model/meshes/ur5/v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
- link shoulder_link: geometry collision mesh filename=/home/mzwang/catkin_ws/src/trajectory_my/model/meshes/ur5/c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; visual mesh filename=/home/mzwang/catkin_ws/src/trajectory_my/model/meshes/ur5/v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
- link upper_arm_link: geometry collision mesh filename=/home/mzwang/catkin_ws/src/trajectory_my/model/meshes/ur5/c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; visual mesh filename=/home/mzwang/catkin_ws/src/trajectory_my/model/meshes/ur5/v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
- link wrist_1_link: geometry collision mesh filename=/home/mzwang/catkin_ws/src/trajectory_my/model/meshes/ur5/c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; visual mesh filename=/home/mzwang/catkin_ws/src/trajectory_my/model/meshes/ur5/v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
- link wrist_2_link: geometry collision mesh filename=/home/mzwang/catkin_ws/src/trajectory_my/model/meshes/ur5/c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; visual mesh filename=/home/mzwang/catkin_ws/src/trajectory_my/model/meshes/ur5/v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
- link wrist_3_link: geometry collision mesh filename=/home/mzwang/catkin_ws/src/trajectory_my/model/meshes/ur5/c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; visual mesh filename=/home/mzwang/catkin_ws/src/trajectory_my/model/meshes/ur5/v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
