Commit message: 4/13 push for discussion

File: model/urdf/pusher.urdf (robot description, URDF)
Before this commit: robot pusher, 4 links, 3 joints
Joints:
- joint base_to_pusher: limit lower=-0.05 upper=0.2 effort=1000.0 velocity=0.5 -> lower=-0.05 upper=0.5 effort=1000.0 velocity=0.5

Commit message: manually calcualted distance&jacobian working

File: model/urdf/pusher.urdf (robot description, URDF)
Before this commit: robot pusher, 4 links, 3 joints
Joints:
- joint base_to_pusher: limit lower=-0.05 upper=0.5 effort=1000.0 velocity=0.5 -> lower=-0.05 upper=1.0 effort=1000.0 velocity=1.0
