Commit message: working for ur1.5

File: model/urdf/ur3e_robot_abs.urdf (robot description, URDF)
Before this commit: robot ur3e, 11 links, 10 joints
Joints:
- joint shoulder_pan_joint: type fixed -> revolute
- joint wrist_2_joint: origin xyz=0.0 0.104 0.0 rpy=0.0 0.0 1.57 -> xyz=0.0 0.104 0.0 rpy=0.0 0.0 0.0; type fixed -> revolute
- joint wrist_3_joint: type fixed -> revolute

Commit message: penalty for slack

File: model/urdf/ur3e_robot_abs.urdf (robot description, URDF)
Before this commit: robot ur3e, 11 links, 10 joints
Joints:
- joint shoulder_pan_joint: type revolute -> fixed
- joint wrist_2_joint: origin xyz=0.0 0.104 0.0 rpy=0.0 0.0 0.0 -> xyz=0.0 0.104 0.0 rpy=0.0 0.0 1.57; type revolute -> fixed
- joint wrist_3_joint: type revolute -> fixed

Commit message: +1

File: model/urdf/ur3e_robot_abs.urdf (robot description, URDF)
Before this commit: robot ur3e, 11 links, 10 joints
Joints:
- joint ee_fixed_joint: origin xyz=0.0 0.092 0.0 rpy=0.0 0.0 1.57079632679 -> xyz=0.0 0.092 0.0 rpy=-1.57079632679 0.0 0.0
