Commit message: change box position in urdf

File: model/urdf/ur3e_robot_box.urdf (robot description, URDF)
Before this commit: robot ur3e, 14 links, 13 joints
Joints:
- joint box_rotate: origin xyz=0 0 0 -> xyz=0 0 0.05

Commit message: multi contact pairs & STC test

File: model/urdf/ur3e_robot_box.urdf (robot description, URDF)
Before this commit: robot ur3e, 14 links, 13 joints
Links:
- added link obj_front; visual box size=0.0001 0.08 0.08
- added link obj_left; visual box size=0.08 0.0001 0.08
- added link obj_right; visual box size=0.08 0.0001 0.08
- link ee_link: geometry collision cylinder length=0.010 radius=0.03; visual sphere radius=0.005
Joints:
- added joint obj_front_link: type fixed, parent box, child obj_front, origin xyz=-0.05 0 0
- added joint obj_left_link: type fixed, parent box, child obj_left, origin xyz=0 0.05 0
- added joint obj_right_link: type fixed, parent box, child obj_right, origin xyz=0 -0.05 0
