Commit message: distance calculation works

File: model/urdf/box.urdf (robot description, URDF)
Before this commit: robot box, 1 links, 0 joints
Links:
- added link obj_front; collision box size=1e-3 0.05 0.05; visual box size=1e-3 0.05 0.05
Joints:
- added joint obj_front_link: type fixed, parent box, child obj_front, origin xyz=-0.025 0 0

Commit message: fix ddq_dv & normal vector for calculating fext

File: model/urdf/box.urdf (robot description, URDF)
Before this commit: robot boxx, 2 links, 1 joints
Links:
- link box: geometry collision box size=0.1 0.1 0.1; visual box size=0.1 0.1 0.1
- link obj_front: geometry collision box size=1e-3 0.1 0.1; visual box size=1e-3 0.1 0.1
Joints:
- joint obj_front_link: origin xyz=-0.025 0 0 -> xyz=-0.05 0 0

Commit message: finding ddq_dq with fext(q)

File: model/urdf/box.urdf (robot description, URDF)
Before this commit: robot boxx, 2 links, 1 joints
Links:
- link box: geometry collision box size=0.05 0.05 0.05; visual box size=0.05 0.05 0.05
- link obj_front: geometry collision box size=1e-3 0.05 0.05; visual box size=1e-3 0.05 0.05
Joints:
- joint obj_front_link: origin xyz=-0.05 0 0 -> xyz=-0.025 0 0

File: model/urdf/ur3e_robot_abs.urdf (robot description, URDF)
Before this commit: robot ur3e, 11 links, 10 joints
Joints:
- joint shoulder_pan_joint: type revolute -> fixed
- joint wrist_2_joint: origin xyz=0.0 0.104 0.0 rpy=0.0 0.0 0.0 -> xyz=0.0 0.104 0.0 rpy=0.0 0.0 1.57; type revolute -> fixed
- joint wrist_3_joint: type revolute -> fixed

Commit message: use fixed contact point

File: model/urdf/box.urdf (robot description, URDF)
Before this commit: robot boxx, 2 links, 1 joints
Links:
- link obj_front: geometry collision sphere radius=1e-6; visual sphere radius=1e-6

Commit message: ur1.5

File: model/urdf/box.urdf (robot description, URDF)
Before this commit: robot boxx, 2 links, 1 joints
Links:
- link obj_front: geometry collision sphere radius=1e-10; visual sphere radius=1e-10

File: model/urdf/ur3e_robot_abs.urdf (robot description, URDF)
Before this commit: robot ur3e, 11 links, 10 joints
Links:
- link ee_link: geometry collision sphere radius=1e-10

Commit message: +3

File: model/urdf/box.urdf (robot description, URDF)
Before this commit: robot boxx, 2 links, 1 joints
Links:
- link box: mass 1 -> 0.6; geometry collision box size=0.1 0.1 0.1; visual box size=0.1 0.1 0.1
- link obj_front: geometry collision box size=0.1 0.1 0.01; visual box size=0.01 0.1 0.1
Joints:
- joint obj_front_link: origin xyz=-0.025 0 0 -> xyz=-0.05 0 0

Commit message: add multi contact sites, not done

File: model/urdf/box.urdf (robot description, URDF)
Before this commit: robot boxx, 2 links, 1 joints
Links:
- added link obj_left; collision box size=0.1 0.01 0.1; visual box size=0.1 0.01 0.1
- added link obj_right; collision box size=0.1 0.01 0.1; visual box size=0.1 0.01 0.1
- link obj_front: geometry collision box size=0.01 0.1 0.1; visual box size=0.01 0.1 0.1
Joints:
- added joint obj_left_link: type fixed, parent box, child obj_left, origin xyz=0 0.05 0
- added joint obj_right_link: type fixed, parent box, child obj_right, origin xyz=0 -0.05 0

Commit message: add the back surface

File: model/urdf/box.urdf (robot description, URDF)
Before this commit: robot boxx, 4 links, 3 joints
Links:
- added link obj_back; collision box size=0.01 0.1 0.1; visual box size=0.01 0.1 0.1
Joints:
- added joint obj_back_link: type fixed, parent box, child obj_back, origin xyz=0.05 0 0
